File: RMR PCB/RMR Electronics.sch (KiCad schematic (older format))
At the start: 19 parts, among them J1 Arduino Power, J2 RPI Power, J3 Mast Servo, J4 RMotor, J5 LMotor, J6 Conn_01x01_Male, J7 LMotor Control, J8 RMotor Control, U1 LD1117S18TR_SOT223, U2 LD1117S18TR_SOT223

Commit message: modified battery power method
Parts:
- gave numbers to parts that had none: 1
Changed lines of the file:
@@
 $EndComp
 $Comp
-L GND #PWR01
+L GND #PWR3
 U 1 1 5B1ABB87
 P 3100 2200
-F 0 "#PWR01" H 3100 1950 50  0001 C CNN
+F 0 "#PWR3" H 3100 1950 50  0001 C CNN
 F 1 "GND" H 3100 2050 50  0000 C CNN
 F 2 "" H 3100 2200 50  0001 C CNN
@@
 $EndComp
 $Comp
-L GND #PWR02
+L GND #PWR4
 U 1 1 5B1ABBCB
 P 3800 3450
-F 0 "#PWR02" H 3800 3200 50  0001 C CNN
+F 0 "#PWR4" H 3800 3200 50  0001 C CNN
 F 1 "GND" H 3800 3300 50  0000 C CNN
 F 2 "" H 3800 3450 50  0001 C CNN
@@
 $EndComp
 $Comp
-L GND #PWR03
+L GND #PWR1
 U 1 1 5B1B3E95
 P 2650 2550
-F 0 "#PWR03" H 2650 2300 50  0001 C CNN
+F 0 "#PWR1" H 2650 2300 50  0001 C CNN
 F 1 "GND" H 2650 2400 50  0000 C CNN
 F 2 "" H 2650 2550 50  0001 C CNN
@@
 $EndComp
 $Comp
-L GND #PWR04
+L GND #PWR5
 U 1 1 5B1B4450
 P 5000 3600
-F 0 "#PWR04" H 5000 3350 50  0001 C CNN
+F 0 "#PWR5" H 5000 3350 50  0001 C CNN
 F 1 "GND" H 5000 3450 50  0000 C CNN
 F 2 "" H 5000 3600 50  0001 C CNN
@@
 $EndComp
 $Comp
-L GND #PWR05
+L GND #PWR6
 U 1 1 5B1B466A
 P 5550 1900
-F 0 "#PWR05" H 5550 1650 50  0001 C CNN
+F 0 "#PWR6" H 5550 1650 50  0001 C CNN
 F 1 "GND" H 5550 1750 50  0000 C CNN
 F 2 "" H 5550 1900 50  0001 C CNN
@@
 	6200 2400 6200 1500
 $Comp
-L GND #PWR07
+L GND #PWR7
 U 1 1 5B3D4DB1
 P 7150 3450
-F 0 "#PWR07" H 7150 3200 50  0001 C CNN
+F 0 "#PWR7" H 7150 3200 50  0001 C CNN
 F 1 "GND" H 7150 3300 50  0000 C CNN
 F 2 "" H 7150 3450 50  0001 C CNN
@@
 	5400 2550 5400 2450
 $Comp
-L PJ-037A J?
+L PJ-037A J9
 U 1 1 5B3E30AA
 P 2350 2950
-F 0 "J?" H 2050 3150 50  0000 L BNN
+F 0 "J9" H 2050 3150 50  0000 L BNN
 F 1 "PJ-037A" H 2049 2750 50  0000 L BNN
 F 2 "CUI_PJ-037A" H 2350 2950 50  0001 L BNN
@@
 $EndComp
 $Comp
-L GND #PWR?
+L GND #PWR2
 U 1 1 5B3E3143
 P 2700 3050
-F 0 "#PWR?" H 2700 2800 50  0001 C CNN
+F 0 "#PWR2" H 2700 2800 50  0001 C CNN
 F 1 "GND" H 2700 2900 50  0000 C CNN
 F 2 "" H 2700 3050 50  0001 C CNN

Commit message: started PCB layout
Parts:
- removed U1, U2: LD1117S18TR_SOT223, TO_SOT_Packages_SMD:SOT-223-3Lead_TabPin2, symbol LD1117S18TR_SOT223
- added U1, U2: AP2204R-5.0, TO_SOT_Packages_SMD:SOT-89-3, symbol AP2204R-5.0
- J9: footprint CUI_PJ-037A -> PJ-037A:CUI_PJ-037A
Connections:
- net GND: now also H1.12 (GND), H1.13 (GND), H1.4 (GND), H1.5 (GND), U1.2 (GND), U2.2 (GND); no longer H1.10 (4A)
- net at C2.1, J2.1 (Pin_1): now also U1.3 (VOUT)
- net at C1.1, C3.1, J1.1 (Pin_1)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: now also U1.1 (VIN), U2.1 (VIN)
- net at C4.1, R1.2: now also U2.3 (VOUT)
- net at C5.1, D1.1 (K), H1.1 (EN)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: now also H1.16 (VCC1), H1.8 (VCC2), H1.9 (EN); no longer H1.15 (3A), H1.2 (1A), H1.7 (2A)
- net at J8.1 (Pin_1): now also H1.2 (1A); no longer H1.3 (1Y)
- net at J8.2 (Pin_2): now also H1.7 (2A); no longer H1.6 (2Y)
- net at J7.1 (Pin_1): now also H1.10 (4A); no longer H1.11 (4Y)
- net at J5.1 (Pin_1): now also H1.11 (4Y); no longer H1.12 (GND)
- net at J5.2 (Pin_2): now also H1.14 (3Y); no longer H1.13 (GND)
- net at J7.2 (Pin_2): now also H1.15 (3A); no longer H1.14 (3Y)
- net at J4.1 (Pin_1): now also H1.3 (1Y); no longer H1.4 (GND)
- net at J4.2 (Pin_2): now also H1.6 (2Y); no longer H1.5 (GND)
Other:
- moved on the sheet: H1, J7

Commit message: reduced  PCB size drastically, outstanding GND copper pour issue
Parts:
- removed J9: PJ-037A, PJ-037A:CUI_PJ-037A, symbol PJ-037A
- added J9: Power In, Pin_Headers:Pin_Header_Straight_1x02_Pitch2.54mm, symbol Conn_01x02_Male
- H1: symbol HBridge -> HBridge-RESCUE-RMR_Electronics
Connections:
- net GND: now also J9.2 (Pin_2)
- net at C1.1, C3.1, J1.1 (Pin_1)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: now also J9.1 (Pin_1)
Changed lines of the file:
@@
 EESchema Schematic File Version 2
+LIBS:RMR Electronics-rescue
 LIBS:power
 LIBS:device
@@
 $EndDescr
 $Comp
-L GND #PWR01
+L GND #PWR3
 U 1 1 5B1ABB87
 P 3100 2200
-F 0 "#PWR01" H 3100 1950 50  0001 C CNN
+F 0 "#PWR3" H 3100 1950 50  0001 C CNN
 F 1 "GND" H 3100 2050 50  0000 C CNN
 F 2 "" H 3100 2200 50  0001 C CNN
@@
 $EndComp
 $Comp
-L GND #PWR02
+L GND #PWR4
 U 1 1 5B1ABBCB
 P 3800 3450
-F 0 "#PWR02" H 3800 3200 50  0001 C CNN
+F 0 "#PWR4" H 3800 3200 50  0001 C CNN
 F 1 "GND" H 3800 3300 50  0000 C CNN
 F 2 "" H 3800 3450 50  0001 C CNN
@@
 $EndComp
 $Comp
-L GND #PWR03
+L GND #PWR1
 U 1 1 5B1B3E95
 P 2650 2550
-F 0 "#PWR03" H 2650 2300 50  0001 C CNN
+F 0 "#PWR1" H 2650 2300 50  0001 C CNN
 F 1 "GND" H 2650 2400 50  0000 C CNN
 F 2 "" H 2650 2550 50  0001 C CNN
@@
 $EndComp
 $Comp
-L GND #PWR04
+L GND #PWR5
 U 1 1 5B1B4450
 P 5000 3600
-F 0 "#PWR04" H 5000 3350 50  0001 C CNN
+F 0 "#PWR5" H 5000 3350 50  0001 C CNN
 F 1 "GND" H 5000 3450 50  0000 C CNN
 F 2 "" H 5000 3600 50  0001 C CNN
@@
 $EndComp
 $Comp
-L GND #PWR05
+L GND #PWR7
 U 1 1 5B1B466A
 P 5550 1900
-F 0 "#PWR05" H 5550 1650 50  0001 C CNN
+F 0 "#PWR7" H 5550 1650 50  0001 C CNN
 F 1 "GND" H 5550 1750 50  0000 C CNN
 F 2 "" H 5550 1900 50  0001 C CNN
@@
 $EndComp
 $Comp
-L HBridge H1
+L HBridge-RESCUE-RMR_Electronics H1
 U 1 1 5B3D44D2
 P 6250 3200
@@
 $EndComp
 $Comp
-L GND #PWR06
+L GND #PWR8
 U 1 1 5B3D4DB1
 P 7150 3250
-F 0 "#PWR06" H 7150 3000 50  0001 C CNN
+F 0 "#PWR8" H 7150 3000 50  0001 C CNN
 F 1 "GND" H 7150 3100 50  0000 C CNN
 F 2 "" H 7150 3250 50  0001 C CNN
@@
 $EndComp
 $Comp
-L PJ-037A J9
-U 1 1 5B3E30AA
-P 2350 2950
-F 0 "J9" H 2050 3150 50  0000 L BNN
-F 1 "PJ-037A" H 2049 2750 50  0000 L BNN
-F 2 "PJ-037A:CUI_PJ-037A" H 2350 2950 50  0001 L BNN
-F 3 "Manufacturer recommendations" H 2350 2950 50  0001 L BNN
-F 4 "CUI INC" H 2350 2950 50  0001 L BNN "Field4"
-	1    2350 2950
-	1    0    0    -1
-$EndComp
-$Comp
-L GND #PWR07
+L GND #PWR2
 U 1 1 5B3E3143
-P 2700 3050
-F 0 "#PWR07" H 2700 2800 50  0001 C CNN
-F 1 "GND" H 2700 2900 50  0000 C CNN
-F 2 "" H 2700 3050 50  0001 C CNN
-F 3 "" H 2700 3050 50  0001 C CNN
-	1    2700 3050
+P 2700 2950
+F 0 "#PWR2" H 2700 2700 50  0001 C CNN
+F 1 "GND" H 2700 2800 50  0000 C CNN
+F 2 "" H 2700 2950 50  0001 C CNN
+F 3 "" H 2700 2950 50  0001 C CNN
+	1    2700 2950
 	0    -1   -1   0
 $EndComp
@@
 	5400 2550 5400 2450
 Wire Wire Line
-	2550 3050 2700 3050
+	2550 2950 2700 2950
 Wire Wire Line
 	5750 3700 5750 3450
@@
 Connection ~ 5600 2850
 $Comp
-L GND #PWR08
+L GND #PWR6
 U 1 1 5B3E75CC
 P 5500 3500
-F 0 "#PWR08" H 5500 3250 50  0001 C CNN
+F 0 "#PWR6" H 5500 3250 50  0001 C CNN
 F 1 "GND" H 5500 3350 50  0000 C CNN
 F 2 "" H 5500 3500 50  0001 C CNN
@@
 	1    0    0    -1
 $EndComp
+$Comp
+L Conn_01x02_Male J9
+U 1 1 5B3E9031
+P 2350 2850
+F 0 "J9" H 2350 2950 50  0000 C CNN
+F 1 "Power In" H 2350 2650 50  0000 C CNN
+F 2 "Pin_Headers:Pin_Header_Straight_1x02_Pitch2.54mm" H 2350 2850 50  0001 C CNN
+F 3 "" H 2350 2850 50  0001 C CNN
+	1    2350 2850
+	1    0    0    -1
+$EndComp

Commit message: Fixed up an issue with the indicator LED
Parts:
- RPI_VRM1: renamed from U1; value AP2204R-5.0 -> RPI VRM
- SIGNAL1: renamed from J6; value Conn_01x01_Male -> SIGNAL
- renumbered J1 to ARD1, J9 to LINE1, J7 to LMI1, J5 to LMO1, U2 to MTR_VRM1, J8 to RMI1, J4 to RMO1, J2 to RPI1, J3 to SERVO1
Connections:
- net GND: now also D1.1 (K)
- net at C4.1, MTR_VRM1.3 (VOUT), R1.2: now also C5.1, H1.1 (EN), H1.16 (VCC1), H1.8 (VCC2), H1.9 (EN), SERVO1.1 (Pin_1)
Changed lines of the file:
@@
 $EndDescr
 $Comp
-L GND #PWR3
+L GND #PWR01
 U 1 1 5B1ABB87
 P 3100 2200
-F 0 "#PWR3" H 3100 1950 50  0001 C CNN
+F 0 "#PWR01" H 3100 1950 50  0001 C CNN
 F 1 "GND" H 3100 2050 50  0000 C CNN
 F 2 "" H 3100 2200 50  0001 C CNN
@@
 $EndComp
 $Comp
-L GND #PWR4
+L GND #PWR02
 U 1 1 5B1ABBCB
 P 3800 3450
-F 0 "#PWR4" H 3800 3200 50  0001 C CNN
+F 0 "#PWR02" H 3800 3200 50  0001 C CNN
 F 1 "GND" H 3800 3300 50  0000 C CNN
 F 2 "" H 3800 3450 50  0001 C CNN
@@
 $EndComp
 $Comp
-L GND #PWR1
+L GND #PWR03
 U 1 1 5B1B3E95
 P 2650 2550
-F 0 "#PWR1" H 2650 2300 50  0001 C CNN
+F 0 "#PWR03" H 2650 2300 50  0001 C CNN
 F 1 "GND" H 2650 2400 50  0000 C CNN
 F 2 "" H 2650 2550 50  0001 C CNN
@@
 $EndComp
 $Comp
-L GND #PWR5
+L GND #PWR04
 U 1 1 5B1B4450
 P 5000 3600
-F 0 "#PWR5" H 5000 3350 50  0001 C CNN
+F 0 "#PWR04" H 5000 3350 50  0001 C CNN
 F 1 "GND" H 5000 3450 50  0000 C CNN
 F 2 "" H 5000 3600 50  0001 C CNN
@@
 $EndComp
 $Comp
-L GND #PWR7
+L GND #PWR05
 U 1 1 5B1B466A
 P 5550 1900
-F 0 "#PWR7" H 5550 1650 50  0001 C CNN
+F 0 "#PWR05" H 5550 1650 50  0001 C CNN
 F 1 "GND" H 5550 1750 50  0000 C CNN
 F 2 "" H 5550 1900 50  0001 C CNN
@@
 $EndComp
 $Comp
-L Conn_01x03_Male J3
+L Conn_01x03_Male SERVO1
 U 1 1 5B3D3D7B
 P 5700 1300
-F 0 "J3" H 5700 1500 50  0000 C CNN
+F 0 "SERVO1" H 5700 1500 50  0000 C CNN
 F 1 "Mast Servo" H 5700 1100 50  0000 C CNN
 F 2 "Pin_Headers:Pin_Header_Straight_1x03_Pitch2.54mm" H 5700 1300 50  0001 C CNN
@@
 $EndComp
 $Comp
-L Conn_01x02_Male J8
+L Conn_01x02_Male RMI1
 U 1 1 5B3D40E6
 P 7200 3800
-F 0 "J8" H 7200 3900 50  0000 C CNN
+F 0 "RMI1" H 7200 3900 50  0000 C CNN
 F 1 "RMotor Control" H 7200 3600 50  0000 C CNN
 F 2 "Pin_Headers:Pin_Header_Straight_1x02_Pitch2.54mm" H 7200 3800 50  0001 C CNN
@@
 $EndComp
 $Comp
-L Conn_01x02_Male J7
+L Conn_01x02_Male LMI1
 U 1 1 5B3D46A6
 P 7250 3050
-F 0 "J7" H 7250 3150 50  0000 C CNN
+F 0 "LMI1" H 7250 3150 50  0000 C CNN
 F 1 "LMotor Control" H 7250 2850 50  0000 C CNN
 F 2 "Pin_Headers:Pin_Header_Straight_1x02_Pitch2.54mm" H 7250 3050 50  0001 C CNN
@@
 $EndComp
 $Comp
-L Conn_01x02_Male J4
+L Conn_01x02_Male RMO1
 U 1 1 5B3D4A9D
 P 6300 1300
-F 0 "J4" H 6300 1400 50  0000 C CNN
+F 0 "RMO1" H 6300 1400 50  0000 C CNN
 F 1 "RMotor" H 6300 1100 50  0000 C CNN
 F 2 "Pin_Headers:Pin_Header_Straight_1x02_Pitch2.54mm" H 6300 1300 50  0001 C CNN
@@
 $EndComp
 $Comp
-L Conn_01x02_Male J5
+L Conn_01x02_Male LMO1
 U 1 1 5B3D4B10
 P 6700 1300
-F 0 "J5" H 6700 1400 50  0000 C CNN
+F 0 "LMO1" H 6700 1400 50  0000 C CNN
 F 1 "LMotor" H 6700 1100 50  0000 C CNN
 F 2 "Pin_Headers:Pin_Header_Straight_1x02_Pitch2.54mm" H 6700 1300 50  0001 C CNN
@@
 $EndComp
 $Comp
-L GND #PWR8
+L GND #PWR06
 U 1 1 5B3D4DB1
-P 7150 3250
-F 0 "#PWR8" H 7150 3000 50  0001 C CNN
-F 1 "GND" H 7150 3100 50  0000 C CNN
-F 2 "" H 7150 3250 50  0001 C CNN
-F 3 "" H 7150 3250 50  0001 C CNN
-	1    7150 3250
+P 7000 3250
+F 0 "#PWR06" H 7000 3000 50  0001 C CNN
+F 1 "GND" H 7000 3100 50  0000 C CNN
+F 2 "" H 7000 3250 50  0001 C CNN
+F 3 "" H 7000 3250 50  0001 C CNN
+	1    7000 3250
 	0    -1   -1   0
 $EndComp
 $Comp
-L Conn_01x01_Male J6
+L Conn_01x01_Male SIGNAL1
 U 1 1 5B3D5099
 P 7200 2250
-F 0 "J6" H 7200 2350 50  0000 C CNN
-F 1 "Conn_01x01_Male" H 7200 2150 50  0000 C CNN
+F 0 "SIGNAL1" H 7200 2350 50  0000 C CNN
+F 1 "SIGNAL" H 7200 2150 50  0000 C CNN
 F 2 "Pin_Headers:Pin_Header_Straight_1x01_Pitch2.54mm" H 7200 2250 50  0001 C CNN
 F 3 "" H 7200 2250 50  0001 C CNN
@@
 $EndComp
 $Comp
-L Conn_01x02_Male J2
+L Conn_01x02_Male RPI1
 U 1 1 5B3D56EC
 P 2900 1950
-F 0 "J2" H 2900 2050 50  0000 C CNN
+F 0 "RPI1" H 2900 2050 50  0000 C CNN
 F 1 "RPI Power" H 2900 1750 50  0000 C CNN
 F 2 "Pin_Headers:Pin_Header_Straight_1x02_Pitch2.54mm" H 2900 1950 50  0001 C CNN
@@
 $EndComp
 $Comp
-L Conn_01x02_Male J1
+L Conn_01x02_Male ARD1
 U 1 1 5B3D578B
 P 2400 2350
-F 0 "J1" H 2400 2450 50  0000 C CNN
+F 0 "ARD1" H 2400 2450 50  0000 C CNN
 F 1 "Arduino Power" H 2400 2150 50  0000 C CNN
 F 2 "Pin_Headers:Pin_Header_Straight_1x02_Pitch2.54mm" H 2400 2350 50  0001 C CNN
@@
 $EndComp
 $Comp
-L GND #PWR2
+L GND #PWR07
 U 1 1 5B3E3143
 P 2700 2950
-F 0 "#PWR2" H 2700 2700 50  0001 C CNN
+F 0 "#PWR07" H 2700 2700 50  0001 C CNN
 F 1 "GND" H 2700 2800 50  0000 C CNN
 F 2 "" H 2700 2950 50  0001 C CNN
@@
 Connection ~ 5850 1750
 Wire Wire Line
-	5400 2100 5850 2100
+	5500 2100 5850 2100
 Wire Wire Line
 	5600 1500 5600 1600
@@
 	5350 2850 5350 2700
 Wire Wire Line
-	5350 2700 5100 2700
+	5100 2700 5500 2700
 Wire Wire Line
 	5100 2700 5100 2550
@@
 	6950 3450 6650 3450
 Wire Wire Line
-	6650 3250 7150 3250
+	6650 3250 7000 3250
 Wire Wire Line
 	6650 3150 6800 3150
@@
 Connection ~ 5600 2850
 $Comp
-L GND #PWR6
+L GND #PWR08
 U 1 1 5B3E75CC
 P 5500 3500
-F 0 "#PWR6" H 5500 3250 50  0001 C CNN
+F 0 "#PWR08" H 5500 3250 50  0001 C CNN
 F 1 "GND" H 5500 3350 50  0000 C CNN
 F 2 "" H 5500 3500 50  0001 C CNN
@@
 	6950 3050 7050 3050
 $Comp
-L AP2204R-5.0 U1
+L AP2204R-5.0 RPI_VRM1
 U 1 1 5B3E7D12
 P 3800 2850
-F 0 "U1" H 3600 2975 50  0000 L CNN
-F 1 "AP2204R-5.0" H 3800 2975 50  0000 L CNN
+F 0 "RPI_VRM1" H 3600 2975 50  0000 L CNN
+F 1 "RPI VRM" H 3600 3050 50  0000 L CNN
 F 2 "TO_SOT_Packages_SMD:SOT-89-3" H 3800 3075 50  0001 C CNN
 F 3 "" H 3800 2850 50  0001 C CNN
@@
 $EndComp
 $Comp
-L AP2204R-5.0 U2
+L AP2204R-5.0 MTR_VRM1
 U 1 1 5B3E7D96
 P 5000 2850
-F 0 "U2" H 4800 2975 50  0000 L CNN
-F 1 "AP2204R-5.0" H 5000 2975 50  0000 L CNN
+F 0 "MTR_VRM1" H 4800 2975 50  0000 L CNN
+F 1 "AP2204R-5.0" H 4800 3050 50  0000 L CNN
 F 2 "TO_SOT_Packages_SMD:SOT-89-3" H 5000 3075 50  0001 C CNN
 F 3 "" H 5000 2850 50  0001 C CNN
@@
 $EndComp
 $Comp
-L Conn_01x02_Male J9
+L Conn_01x02_Male LINE1
 U 1 1 5B3E9031
 P 2350 2850
-F 0 "J9" H 2350 2950 50  0000 C CNN
+F 0 "LINE1" H 2350 2950 50  0000 C CNN
 F 1 "Power In" H 2350 2650 50  0000 C CNN
 F 2 "Pin_Headers:Pin_Header_Straight_1x02_Pitch2.54mm" H 2350 2850 50  0001 C CNN
@@
 	1    0    0    -1
 $EndComp
+Connection ~ 5350 2700
+$Comp
+L GND #PWR09
+U 1 1 5B3F777A
+P 5400 2100
+F 0 "#PWR09" H 5400 1850 50  0001 C CNN
+F 1 "GND" H 5400 1950 50  0000 C CNN
+F 2 "" H 5400 2100 50  0001 C CNN
+F 3 "" H 5400 2100 50  0001 C CNN
+	1    5400 2100
+	-1   0    0    1
+$EndComp
+Wire Wire Line
+	5500 2700 5500 2100
 $EndSCHEMATC
